File: CYM1A113.kicad_pcb (KiCad board)
At the start: 4 copper layers, 59 x 33.8 mm, 128 parts, among them IC1 MIC803-29D2VC3, IC2 STM32F427VIT6, IC5 TPS61043, IC6 XC6210B332PR, K1 DX07B024XJ1R1300, K3 ATTEND_112J-TDAR-R01, K4 DF37NB-24DS-0.4V, K5 SWD, K6 DF37NB-10DS-0.4V, T1 DMG3415U-7, T2 DMG3415U-7, X1 CTS406 8MHz

Commit message: Routing improvements.
Move the display traces away from the first inner layer to
keep it as an unbroken ground plane. This eliminates most of the
jumper traces, still using the first inner layer as reference plane
for display and touchscreen signal.
Routing:
- net VCC-2: track 89.3 -> 119.8 mm
- net /CC2: track 9.04 -> 8.54 mm
- net Net-(IC2-Pad61): vias 3 -> 2
- net Net-(IC2-Pad62): vias 3 -> 2
- net Net-(IC2-Pad59): vias 3 -> 2
- net Net-(IC2-Pad58): vias 3 -> 2
- net /LEDK: vias 3 -> 2
- net /LEDA: vias 3 -> 2
